Commit message: Update links, joints, and args

File: dolly_description/models/dolly.xacro (robot description, xacro)
@@ -1,25 +1,17 @@
 <?xml version="1.0" ?>
 <robot name="dolly" xmlns:xacro="http://www.ros.org/wiki/xacro">
-  <xacro:arg name="sim_gazebo_classic" default="true" />
-  <xacro:arg name="sim_ignition_classic" default="false" />
+  <xacro:arg name="sim_gazebo_classic" default="$(optenv SIM_GAZEBO_CLASSIC)" />
+  <xacro:arg name="sim_ignition" default="$(optenv SIM_IGNITION)" />
   <link name='chassis'>
     <inertial>
-      <mass>1.0</mass>
-      <inertia>
-        <ixx>0.0227</ixx>
-        <ixy>0</ixy>
-        <ixz>0</ixz>
-        <iyy>0.0852</iyy>
-        <iyz>0</iyz>
-        <izz>0.1041</izz>
-      </inertia>
-    </inertial>
-    <visual name='visual'>
-      <geometry>
-        <box>
-          <size>1.0 0.5 0.15</size>
-        </box>
-      </geometry>
-      <material>
+      <mass value="1"/>
+      <origin rpy="0 0 0" xyz="0 0 0."/>
+      <inertia ixx="0.0277" ixy="0" ixz="0" iyy="0.0852" iyz="0" izz="0.1041"/>
+    </inertial>
+    <visual name='visual'>
+      <geometry>
+          <box size="1.0 0.5 0.15"/>
+      </geometry>
+      <material name='chassis_material'>
         <script>
           <uri>model://dolly/materials/scripts</uri>
@@ -32,11 +24,8 @@
       <pose>0 0 0.08 0 0 0.24</pose>
       <geometry>
-        <mesh>
-          <uri>model://cardboard_box/meshes/cardboard_box.dae</uri>
-          <scale>1.25931896 1.007455168 0.755591376</scale>
-        </mesh>
-      </geometry>
-    </visual>
-    <xacro:if value="$(sim_gazebo_classic)">
+          <mesh filename="model://cardboard_box/meshes/cardboard_box.dae" scale="1.25931896 1.007455168 0.755591376" />
+      </geometry>
+    </visual>
+    <xacro:if value="$(arg sim_gazebo_classic)">
       <sensor name="sensor_ray" type="ray">
         <pose>0.5 0 0 0 0 0</pose>
@@ -67,5 +56,5 @@
       </sensor>
     </xacro:if>
-    <xacro:if value="$(sim_ignition)">
+    <xacro:if value="$(arg sim_ignition)">
       <sensor name="sensor_ray" type="gpu_lidar">
         <pose>0.5 0 0 0 0 0</pose>
@@ -94,21 +83,12 @@
     <pose>-0.3 0 -0.125 0 0 0</pose>
     <inertial>
-      <mass>0.0415553</mass>
-      <inertia>
-        <ixx>7.97741e-05</ixx>
-        <ixy>0</ixy>
-        <ixz>0</ixz>
-        <iyy>7.97741e-05</iyy>
-        <iyz>0</iyz>
-        <izz>7.97741e-05</izz>
-      </inertia>
-    </inertial>
-    <visual name='visual'>
-      <geometry>
-        <sphere>
-          <radius>0.1</radius>
-        </sphere>
-      </geometry>
-      <material>
+      <mass value= "0.0415553"/>
+      <inertia ixx="7.97741e-05" ixy="0" ixz="0" iyy="7.97741e-05" iyz="0" izz="7.97741e-05"/>
+    </inertial>
+    <visual name='visual'>
+      <geometry>
+        <sphere radius="0.1"/>
+      </geometry>
+      <material name="caster_material">
         <diffuse>0.5 0.5 0.5 1</diffuse>
         <ambient>0 0 0 1</ambient>
@@ -119,7 +99,5 @@
     <collision name='collision'>
       <geometry>
-        <sphere>
-          <radius>0.1</radius>
-        </sphere>
+        <sphere radius="0.1"/>
       </geometry>
       <surface>
@@ -148,22 +126,12 @@
     <pose>0.3 0.3 -0.075 -1.5707 0 0</pose>
     <inertial>
-      <mass>0.5</mass>
-      <inertia>
-        <ixx>0.0029</ixx>
-        <ixy>0</ixy>
-        <ixz>0</ixz>
-        <iyy>0.0029</iyy>
-        <iyz>0</iyz>
-        <izz>0.0056</izz>
-      </inertia>
-    </inertial>
-    <visual name='visual'>
-      <geometry>
-        <cylinder>
-          <radius>0.15</radius>
-          <length>0.05</length>
-        </cylinder>
-      </geometry>
-      <material>
+      <mass value= "0.5"/>
+      <inertia ixx="0.0029" ixy="0" ixz="0" iyy="0.0029" iyz="0" izz="0.0056" />
+    </inertial>
+    <visual name='visual'>
+      <geometry>
+        <cylinder radius="0.15" length="0.05"/>
+      </geometry>
+      <material name="left_wheel_material">
         <diffuse>0.5 0.5 0.5 1</diffuse>
         <ambient>0 0 0 1</ambient>
@@ -174,7 +142,5 @@
     <collision name='collision'>
       <geometry>
-        <sphere>
-          <radius>0.15</radius>
-        </sphere>
+        <sphere radius="0.1"/>
       </geometry>
       <surface>
@@ -203,22 +169,12 @@
     <pose>0.3 -0.3 -0.075 -1.5707 0 0</pose>
     <inertial>
-      <mass>0.5</mass>
-      <inertia>
-        <ixx>0.0029</ixx>
-        <ixy>0</ixy>
-        <ixz>0</ixz>
-        <iyy>0.0029</iyy>
-        <iyz>0</iyz>
-        <izz>0.0056</izz>
-      </inertia>
-    </inertial>
-    <visual name='visual'>
-      <geometry>
-        <cylinder>
-          <radius>0.15</radius>
-          <length>0.05</length>
-        </cylinder>
-      </geometry>
-      <material>
+      <mass value= "0.5"/>
+      <inertia ixx="0.0029" ixy="0" ixz="0" iyy="0.0029" iyz="0" izz="0.0056" />
+    </inertial>
+    <visual name='visual'>
+      <geometry>
+        <cylinder radius="0.15" length="0.05"/>
+      </geometry>
+      <material name="right_wheel_material">
         <diffuse>0.5 0.5 0.5 1</diffuse>
         <ambient>0 0 0 1</ambient>
@@ -229,7 +185,5 @@
     <collision name='collision'>
       <geometry>
-        <sphere>
-          <radius>0.15</radius>
-        </sphere>
+        <sphere radius="0.1"/>
       </geometry>
       <surface>
@@ -258,23 +212,13 @@
     <pose>-0.52 0 0 -1.6 0 0</pose>
     <inertial>
-      <mass>0.0254232</mass>
-      <inertia>
-        <ixx>1.528e-05</ixx>
-        <ixy>0</ixy>
-        <ixz>0</ixz>
-        <iyy>1.528e-05</iyy>
-        <iyz>0</iyz>
-        <izz>3.45e-06</izz>
-      </inertia>
+      <mass value="0.0254232" />
+      <inertia ixx="1.528e-05" ixy="0" ixz="0" iyy="1.528e-05" iyz="0" izz="3.45e-06" />
       <pose frame=''>0 0 -0.04 0 -0 0</pose>
     </inertial>
     <visual name='visual'>
       <geometry>
-        <cylinder>
-          <radius>0.016468</radius>
-          <length>0.08</length>
-        </cylinder>
-      </geometry>
-      <material>
+        <cylinder radius="0.016468" length="0.08"/>
+      </geometry>
+      <material name="tail_material">
         <script>
           <uri>model://dolly/materials/scripts</uri>
@@ -286,42 +230,31 @@
   </link>
   <joint name='left_wheel_joint' type='revolute'>
-    <parent>chassis</parent>
-    <child>left_wheel</child>
+    <parent link="chassis"/>
+    <child link="left_wheel"/>
+    <limit effort="10" velocity="10"/>
     <axis>
       <xyz>0 0 1</xyz>
-      <limit>
-        <lower>-1.79769e+308</lower>
-        <upper>1.79769e+308</upper>
-      </limit>
     </axis>
   </joint>
   <joint name='right_wheel_joint' type='revolute'>
-    <parent>chassis</parent>
-    <child>right_wheel</child>
+    <parent link="chassis"/>
+    <child link="right_wheel"/>
+    <limit effort="10" velocity="10"/>
     <axis>
       <xyz>0 0 1</xyz>
-      <limit>
-        <lower>-1.79769e+308</lower>
-        <upper>1.79769e+308</upper>
-      </limit>
     </axis>
   </joint>
-  <joint name='caster_wheel' type='ball'>
-    <parent>chassis</parent>
-    <child>caster</child>
+  <joint name='caster_wheel' type='fixed'>
+    <parent link="chassis"/>
+    <child link="caster"/>
   </joint>
   <joint name='tail_joint' type='revolute'>
-    <parent>chassis</parent>
-    <child>tail</child>
+    <parent link="chassis"/>
+    <child link="tail"/>
     <pose>0 0 0.04 0 -0 0</pose>
+    <limit lower="-1.79769e+308" upper="1.79769e+308" effort="-1" velocity="-1" />
     <axis>
       <xyz>1 0 0</xyz>
       <use_parent_model_frame>0</use_parent_model_frame>
-      <limit>
-        <lower>-1.79769e+308</lower>
-        <upper>1.79769e+308</upper>
-        <effort>-1</effort>
-        <velocity>-1</velocity>
-      </limit>
       <dynamics>
         <spring_reference>0</spring_reference>
@@ -344,5 +277,5 @@
     </physics>
   </joint>
-  <xacro:if value="$(sim_gazebo_classic)">
+  <xacro:if value="$(arg sim_gazebo_classic)">
     <gazebo>
       <plugin name='diff_drive' filename='libgazebo_ros_diff_drive.so'>
@@ -367,5 +300,5 @@
     </gazebo>
   </xacro:if>
-  <xacro:if value="$(sim_ignition)">
+  <xacro:if value="$(arg sim_ignition)">
     <gazebo>
       <plugin

Commit message: Move box and laser to new links and update coords

File: dolly_description/models/dolly.xacro (robot description, xacro)
@@ -3,5 +3,5 @@
   <xacro:arg name="sim_gazebo_classic" default="$(optenv SIM_GAZEBO_CLASSIC)" />
   <xacro:arg name="sim_ignition" default="$(optenv SIM_IGNITION)" />
-  <link name='chassis'>
+  <link name="chassis">
     <inertial>
       <mass value="1"/>
@@ -9,5 +9,5 @@
       <inertia ixx="0.0277" ixy="0" ixz="0" iyy="0.0852" iyz="0" izz="0.1041"/>
     </inertial>
-    <visual name='visual'>
+    <visual>
       <geometry>
           <box size="1.0 0.5 0.15"/>
@@ -21,4 +21,11 @@
       </material>
     </visual>
+  </link>
+  <link name="box">
+    <inertial>
+      <mass value="0"/>
+      <origin rpy="0 0 0" xyz="0 0 0."/>
+      <inertia ixx="0" ixy="0" ixz="0" iyy="0" iyz="0" izz="0"/>
+    </inertial>
     <visual name="box">
       <pose>0 0 0.08 0 0 0.24</pose>
@@ -27,5 +34,20 @@
       </geometry>
     </visual>
-    <xacro:if value="$(arg sim_gazebo_classic)">
+  </link>
+  <joint name='box_joint' type='fixed'>
+    <origin xyz="0 0 0.08" rpy="0 0 24"/>
+    <parent link="chassis"/>
+    <child link="box"/>
+    <axis xyz="0 0 1" />
+  </joint>
+  <link name="laser_sensor"/>
+  <joint name='laser_sensor_joint' type='fixed'>
+    <origin xyz="0.5 0 0" rpy="0 0 0"/>
+    <parent link="chassis"/>
+    <child link="laser_sensor"/>
+    <axis xyz="0 0 1" />
+  </joint>
+  <xacro:if value="$(arg sim_gazebo_classic)">
+    <gazebo reference="laser_sensor">
       <sensor name="sensor_ray" type="ray">
         <pose>0.5 0 0 0 0 0</pose>
@@ -55,6 +77,8 @@
         </plugin>
       </sensor>
-    </xacro:if>
-    <xacro:if value="$(arg sim_ignition)">
+    </gazebo>
+  </xacro:if>
+  <xacro:if value="$(arg sim_ignition)">
+    <gazebo reference="laser_sensor">
       <sensor name="sensor_ray" type="gpu_lidar">
         <pose>0.5 0 0 0 0 0</pose>
@@ -78,8 +102,7 @@
         <update_rate>100.0</update_rate>
       </sensor>
-    </xacro:if>
-  </link>
+    </gazebo>
+  </xacro:if>
   <link name='caster'>
-    <pose>-0.3 0 -0.125 0 0 0</pose>
     <inertial>
       <mass value= "0.0415553"/>
@@ -124,5 +147,4 @@
   </link>
   <link name='left_wheel'>
-    <pose>0.3 0.3 -0.075 -1.5707 0 0</pose>
     <inertial>
       <mass value= "0.5"/>
@@ -142,5 +164,5 @@
     <collision name='collision'>
       <geometry>
-        <sphere radius="0.1"/>
+        <cylinder radius="0.15" length="0.05"/>
       </geometry>
       <surface>
@@ -185,5 +207,5 @@
     <collision name='collision'>
       <geometry>
-        <sphere radius="0.1"/>
+        <cylinder radius="0.15" length="0.05"/>
       </geometry>
       <surface>
@@ -210,5 +232,4 @@
   </link>
   <link name='tail'>
-    <pose>-0.52 0 0 -1.6 0 0</pose>
     <inertial>
       <mass value="0.0254232" />
@@ -230,20 +251,19 @@
   </link>
   <joint name='left_wheel_joint' type='revolute'>
+    <origin xyz="0.3 0.3 -0.075" rpy="-1.5707 0 0"/>
     <parent link="chassis"/>
     <child link="left_wheel"/>
     <limit effort="10" velocity="10"/>
-    <axis>
-      <xyz>0 0 1</xyz>
-    </axis>
+    <axis xyz="0 0 1" />
   </joint>
   <joint name='right_wheel_joint' type='revolute'>
+    <origin xyz="0.3 -0.3 -0.075" rpy="-1.5707 0 0"/>
     <parent link="chassis"/>
     <child link="right_wheel"/>
     <limit effort="10" velocity="10"/>
-    <axis>
-      <xyz>0 0 1</xyz>
-    </axis>
+    <axis xyz="0 0 1" />
   </joint>
   <joint name='caster_wheel' type='fixed'>
+    <origin xyz="-0.3 0 -0.125" rpy="0 0 0"/>
     <parent link="chassis"/>
     <child link="caster"/>
@@ -252,5 +272,5 @@
     <parent link="chassis"/>
     <child link="tail"/>
-    <pose>0 0 0.04 0 -0 0</pose>
+    <origin xyz="-0.52 0 0.04" rpy="-1.6 0 0"/>
     <limit lower="-1.79769e+308" upper="1.79769e+308" effort="-1" velocity="-1" />
     <axis>
@@ -316,3 +336,12 @@
     </gazebo>
   </xacro:if>
+  <gazebo reference="chassis">
+    <material>
+      <script>
+        <uri>model://dolly/materials/scripts</uri>
+        <uri>model://dolly/materials/textures</uri>
+        <name>aruco_tag_0</name>
+      </script>
+    </material>
+  </gazebo>
 </robot>

Commit message: Change wheel joint typte

File: dolly_description/models/dolly.xacro (robot description, xacro)
@@ -250,16 +250,18 @@
     </visual>
   </link>
-  <joint name='left_wheel_joint' type='revolute'>
+  <joint name='left_wheel_joint' type='continuous'>
     <origin xyz="0.3 0.3 -0.075" rpy="-1.5707 0 0"/>
     <parent link="chassis"/>
     <child link="left_wheel"/>
     <limit effort="10" velocity="10"/>
+    <joint_properties damping="1.0" friction="1.0"/>
     <axis xyz="0 0 1" />
   </joint>
-  <joint name='right_wheel_joint' type='revolute'>
+  <joint name='right_wheel_joint' type='continuous'>
     <origin xyz="0.3 -0.3 -0.075" rpy="-1.5707 0 0"/>
     <parent link="chassis"/>
     <child link="right_wheel"/>
     <limit effort="10" velocity="10"/>
+    <joint_properties damping="1.0" friction="1.0"/>
     <axis xyz="0 0 1" />
   </joint>
